File: board_kicad/main/board.kicad_pcb (KiCad board)
At the start: 2 copper layers, 68.6 x 53.3 mm, 42 parts, among them J1 Conn_01x02, J20 Conn_01x02, J30 Conn_01x03, J40 RJ45, Q20 IRLM5203 (PMOS_GSD), Q21 IRLM5203 (PMOS_GSD), U1 Arduino_Nano_Every, U20 TPS259630, U30 ADUM1301, U31 MAX487E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

Commit message: extended, improved and finished circuits and boards
also added PDF and renders of shematic/board

INFO: The Displays Library is not included and can be found at
      https://github.com/jonolt/KiCad_lib_EA-Dispaly
Parts:
- added D1: LED, LED_SMD:LED_0805_2012Metric, F.Cu at (110.6, 106.8)
- added D2: LED, LED_SMD:LED_0805_2012Metric, F.Cu at (110.6, 104.3)
- added D30: LED, LED_SMD:LED_0805_2012Metric, F.Cu at (144.5, 111.8)
- added D31: LED, LED_SMD:LED_0805_2012Metric, F.Cu at (144.4, 114.3)
- added R1: 270, Resistor_SMD:R_0805_2012Metric, F.Cu at (115.6, 110.6)
- added R2: 270, Resistor_SMD:R_0805_2012Metric, F.Cu at (115.6, 112.5)
- added R3: R, Resistor_SMD:R_0805_2012Metric, F.Cu at (98.6, 79.0)
- added R33: 270, Resistor_SMD:R_0805_2012Metric, F.Cu at (148.3, 111.8)
- added R34: 270, Resistor_SMD:R_0805_2012Metric, F.Cu at (148.3, 114.3)
- added R4: R, Resistor_SMD:R_0805_2012Metric, F.Cu at (102.0, 79.0)
- added U2: 74LVC2G34, Package_TO_SOT_SMD:SOT-23-6, F.Cu at (111.6, 111.6)
- added U33: 74LVC2G34, Package_TO_SOT_SMD:SOT-23-6, F.Cu at (148.0, 118.7)
- C21: footprint Capacitor_Tantalum_SMD:CP_EIA-3528-15_AVX-H -> Capacitor_SMD:C_0805_2012Metric
- D21: value STPS1L30AFN -> BAT54J; footprint Diode_SMD:D_SMA -> Diode_SMD:D_SOD-323F
- U32: footprint my_lib:SIP7-1-2-4-6 -> project:SIP7-1-2-4-6
- moved J1 5.59 mm to (154.9, 83.8), turned to 0 degrees
- moved D24 4.13 mm to (127.2, 123.8), turned to 0 degrees
- moved C21 3.66 mm to (135.6, 118.1)
- moved D21 2.08 mm to (133.6, 118.1)
- moved D23 1.58 mm to (127.2, 121.3), turned to 0 degrees
- moved R21 0.97 mm to (111.1, 119.4)
- moved R27 0.76 mm to (122.2, 122.8)
- moved D22 0.64 mm to (129.0, 118.1)
- moved R22 0.63 mm to (111.1, 115.6)
- moved JP1 0.38 mm to (154.9, 81.4)
- moved JP2 0.38 mm to (152.4, 81.4)
- moved C20 0.30 mm to (114.3, 115.6)
Routing:
- net /ISO_+5V: track 65.0 -> 96.5 mm
- net /DMX+: track 22.1 -> 42.1 mm, vias 0 -> 1
- net /SDA: track 36.8 -> 55.6 mm, vias 0 -> 2
- net /SCL: track 35.5 -> 50.4 mm, vias 0 -> 1
- net /DMX-: track 22.1 -> 34.1 mm
- net Net-(D2-Pad2): track 0.00 -> 10.9 mm
- net Net-(D30-Pad2): track 0.00 -> 9.36 mm
- net GND: track 52.5 -> 61.2 mm, vias 6 -> 7
- net Net-(D31-Pad2): track 0.00 -> 7.24 mm
- net /ISO_GND: track 89.1 -> 96.2 mm
- net Net-(D1-Pad2): track 0.00 -> 6.36 mm
- net Net-(D24-Pad1): track 8.53 -> 3.85 mm
- net +5V: track 146.1 -> 150.2 mm, vias 3 -> 4
- net /A0-CUR: track 64.0 -> 60.5 mm
- net /~RESET: track 96.9 -> 93.9 mm
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Other:
- net class pwr: clearance 0.4 -> 0.2
- board text added: "(Shield)"
- board text added: "+"
- board text added: "-"
- board text added: "08/2020"
- board text added: "5V"
- board text added: "A0-CUR"
- board text added: "DMX"
- board text added: "I2C"
- board text added: "I2C PULLUP"
- board text added: "NanoE-DMX"
- board text added: "POWER SOURCE"
- board text added: "SCL"
- board text added: "SDA"
- board text added: "TX RX EXTERN"
- board text added: "VIN"
- board text added: "~FLT"
