File: board_kicad/NanoE-DMX/board.kicad_pcb (KiCad board)
At the start: 2 copper layers, 68.6 x 53.3 mm, 56 parts, among them J1 Conn_01x02, J20 Conn_01x02, J30 Conn_01x03, J40 Conn_01x04, Q20 IRLM5203 (PMOS_GSD), Q21 IRLM5203 (PMOS_GSD), U1 Arduino_Nano_Every, U2 74LVC2G34, U20 TPS259630, U30 ADUM1301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

Commit message: minor cleanup
Other:
- board text added: "RX"
- board text added: "TX"
- board text removed: "RX(-)"
- board text removed: "TX(+)"
